Commit message: Replace hardcoded absolute paths with portable placeholders and package:// URIs

File: src/control/mc_rtc_controller/urdf/harambe_mc_rtc.urdf (robot description, URDF)
Before this commit: robot harambe_full_robot, 66 links, 65 joints
Links:
- link left_hand_base_link: geometry collision box size=0.0125 0.0111 0.0089; collision box size=0.0125 0.0111 0.0089
- link left_index_intermediate: geometry collision box size=0.014 0.042 0.010; visual mesh filename=package://hand_description/meshes/inspire_hand/visual/left_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
- link left_index_proximal: geometry collision box size=0.014 0.032 0.012; visual mesh filename=package://hand_description/meshes/inspire_hand/visual/left_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
- link left_middle_intermediate: geometry collision box size=0.014 0.046 0.010; visual mesh filename=package://hand_description/meshes/inspire_hand/visual/left_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
- link left_middle_proximal: geometry collision box size=0.014 0.032 0.012; visual mesh filename=package://hand_description/meshes/inspire_hand/visual/left_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
- link left_pinky_intermediate: geometry collision box size=0.014 0.034 0.010; visual mesh filename=package://hand_description/meshes/inspire_hand/visual/left_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
- link left_pinky_proximal: geometry collision box size=0.014 0.032 0.012; visual mesh filename=package://hand_description/meshes/inspire_hand/visual/left_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
- link left_ring_intermediate: geometry collision box size=0.014 0.042 0.010; visual mesh filename=package://hand_description/meshes/inspire_hand/visual/left_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
- link left_ring_proximal: geometry collision box size=0.014 0.032 0.012; visual mesh filename=package://hand_description/meshes/inspire_hand/visual/left_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
- link left_thumb_distal: geometry collision box size=0.024 0.016 0.012; visual mesh filename=package://hand_description/meshes/inspire_hand/visual/left_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
- link left_thumb_intermediate: geometry collision box size=0.025 0.014 0.014; visual mesh filename=package://hand_description/meshes/inspire_hand/visual/left_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
- link left_thumb_proximal: geometry collision box size=0.050 0.030 0.016; visual mesh filename=package://hand_description/meshes/inspire_hand/visual/left_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
- link left_thumb_proximal_base: geometry collision box size=0.015 0.012 0.014; visual mesh filename=package://hand_description/meshes/inspire_hand/visual/left_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
- link pelvis_imu_sensor: geometry collision mesh filename=package://imu_description/meshes/low_res_bno055_imu.stl; visual mesh filename=package://imu_description/meshes/low_res_bno055_imu.stl
- link right_hand_base_link: geometry collision box size=0.0125 0.0111 0.0089; collision box size=0.0125 0.0111 0.0089
- link right_index_intermediate: geometry collision box size=0.014 0.042 0.010; visual mesh filename=package://hand_description/meshes/inspire_hand/visual/right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
- link right_index_proximal: geometry collision box size=0.014 0.032 0.012; visual mesh filename=package://hand_description/meshes/inspire_hand/visual/right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
- link right_middle_intermediate: geometry collision box size=0.014 0.046 0.010; visual mesh filename=package://hand_description/meshes/inspire_hand/visual/right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
- link right_middle_proximal: geometry collision box size=0.014 0.032 0.012; visual mesh filename=package://hand_description/meshes/inspire_hand/visual/right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
- link right_pinky_intermediate: geometry collision box size=0.014 0.034 0.010; visual mesh filename=package://hand_description/meshes/inspire_hand/visual/right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
- link right_pinky_proximal: geometry collision box size=0.014 0.032 0.012; visual mesh filename=package://hand_description/meshes/inspire_hand/visual/right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
- link right_ring_intermediate: geometry collision box size=0.014 0.042 0.010; visual mesh filename=package://hand_description/meshes/inspire_hand/visual/right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
- link right_ring_proximal: geometry collision box size=0.014 0.032 0.012; visual mesh filename=package://hand_description/meshes/inspire_hand/visual/right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
- link right_thumb_distal: geometry collision box size=0.024 0.016 0.012; visual mesh filename=package://hand_description/meshes/inspire_hand/visual/right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
- link right_thumb_intermediate: geometry collision box size=0.025 0.014 0.014; visual mesh filename=package://hand_description/meshes/inspire_hand/visual/right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
- link right_thumb_proximal: geometry collision box size=0.050 0.030 0.016; visual mesh filename=package://hand_description/meshes/inspire_hand/visual/right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
- link right_thumb_proximal_base: geometry collision box size=0.015 0.012 0.014; visual mesh filename=package://hand_description/meshes/inspire_hand/visual/right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
- link torso_imu_sensor: geometry collision mesh filename=package://imu_description/meshes/low_res_bno055_imu.stl; visual mesh filename=package://imu_description/meshes/low_res_bno055_imu.stl
- link urdf_ankle_assembly: geometry collision mesh filename=package://full_robot_description/meshes/collision/urdf_ankl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; visual mesh filename=package://full_robot_description/meshes/visual/urdf_ankle_a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
- link urdf_ankle_assembly_2: geometry collision mesh filename=package://full_robot_description/meshes/collision/urdf_ankl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; visual mesh filename=package://full_robot_description/meshes/visual/urdf_ankle_a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
- link urdf_base: geometry collision mesh filename=package://full_robot_description/meshes/collision/b_base.stl; collision mesh filename=package://full_robot_description/meshes/collision/f_base.stl
- link urdf_foot_assembly: geometry collision mesh filename=package://full_robot_description/meshes/collision/urdf_foot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; visual mesh filename=package://full_robot_description/meshes/visual/urdf_foot_as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
- link urdf_foot_assembly_2: geometry collision mesh filename=package://full_robot_description/meshes/collision/urdf_foot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; visual mesh filename=package://full_robot_description/meshes/visual/urdf_foot_as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
- link urdf_hip_assembly: geometry collision mesh filename=package://full_robot_description/meshes/collision/hip.stl; visual mesh filename=package://full_robot_description/meshes/visual/hip.stl
- link urdf_hip_assembly_2: geometry collision mesh filename=package://full_robot_description/meshes/collision/hip.stl; visual mesh filename=package://full_robot_description/meshes/visual/hip.stl
- link urdf_l_elbow_assembly: geometry collision mesh filename=package://full_robot_description/meshes/collision/urdf_l_el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; visual mesh filename=package://full_robot_description/meshes/visual/stator_x6_p2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
- link urdf_l_lower_forearm_assembly: geometry collision mesh filename=package://full_robot_description/meshes/collision/urdf_l_lo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; visual mesh filename=package://full_robot_description/meshes/visual/stator_x4_p3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
- link urdf_l_shoulder_assembly: geometry collision mesh filename=package://full_robot_description/meshes/collision/l_shoulde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; visual mesh filename=package://full_robot_description/meshes/visual/l_shoulder.s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
- link urdf_l_tibia_assembly: geometry collision mesh filename=package://full_robot_description/meshes/collision/urdf_l_ti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; visual mesh filename=package://full_robot_description/meshes/visual/m6_threaded_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
- link urdf_l_upper_arm_assembly: geometry collision mesh filename=package://full_robot_description/meshes/collision/urdf_l_up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; visual mesh filename=package://full_robot_description/meshes/visual/stator_x4_p3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
- link urdf_l_upper_femur_assembly: geometry collision mesh filename=package://full_robot_description/meshes/collision/l_upper_f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; visual mesh filename=package://full_robot_description/meshes/visual/l_upper_femu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
- link urdf_l_upper_forearm_assembly: geometry collision mesh filename=package://full_robot_description/meshes/collision/urdf_l_up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; visual mesh filename=package://full_robot_description/meshes/visual/stator_x4_p3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
- link urdf_l_wrist_assembly: geometry collision mesh filename=package://full_robot_description/meshes/collision/l_wrist.s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; visual mesh filename=package://full_robot_description/meshes/visual/l_wrist.stl
- link urdf_lower_femur_assembly: geometry collision mesh filename=package://full_robot_description/meshes/collision/lower_fem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; visual mesh filename=package://full_robot_description/meshes/visual/lower_femur.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
- link urdf_lower_femur_assembly_2: geometry collision mesh filename=package://full_robot_description/meshes/collision/lower_fem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; visual mesh filename=package://full_robot_description/meshes/visual/lower_femur.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
- link urdf_r_elbow_assembly: geometry collision mesh filename=package://full_robot_description/meshes/collision/r_elbow.s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; visual mesh filename=package://full_robot_description/meshes/visual/r_elbow.stl
- link urdf_r_lower_forearm_assembly: geometry collision mesh filename=package://full_robot_description/meshes/collision/r_lower_f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; visual mesh filename=package://full_robot_description/meshes/visual/r_lower_fore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
- link urdf_r_shoulder_assembly: geometry collision mesh filename=package://full_robot_description/meshes/collision/r_shoulde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; visual mesh filename=package://full_robot_description/meshes/visual/r_shoulder.s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
- link urdf_r_tibia_assembly: geometry collision mesh filename=package://full_robot_description/meshes/collision/urdf_r_ti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; visual mesh filename=package://full_robot_description/meshes/visual/m6_threaded_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
- link urdf_r_upper_arm_assembly: geometry collision mesh filename=package://full_robot_description/meshes/collision/r_upper_a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; visual mesh filename=package://full_robot_description/meshes/visual/r_upper_arm.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
- link urdf_r_upper_femur_assemby: geometry collision mesh filename=package://full_robot_description/meshes/collision/r_upper_f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; visual mesh filename=package://full_robot_description/meshes/visual/r_upper_femu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
- link urdf_r_upper_forearm_assembly: geometry collision mesh filename=package://full_robot_description/meshes/collision/r_upper_f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; visual mesh filename=package://full_robot_description/meshes/visual/r_upper_fore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
- link urdf_r_wrist_assembly: geometry collision mesh filename=package://full_robot_description/meshes/collision/r_wrist.s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; visual mesh filename=package://full_robot_description/meshes/visual/r_wrist.stl
- link urdf_simplified_torso: geometry collision mesh filename=package://full_robot_description/meshes/collision/head.stl; collision mesh filename=package://full_robot_description/meshes/collision/urdf_simp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

Commit message: partioal don walking controller

File: src/control/mc_rtc_controller/urdf/harambe_mc_rtc.urdf (robot description, URDF)
Before this commit: robot harambe_full_robot, 66 links, 65 joints
Joints:
- joint left_ankle_pitch_joint_X4: limit lower=-0.79 upper=0.79 effort=10.5 velocity=8.69 -> lower=-0.79 upper=0.79 effort=96.6 velocity=8.69
- joint left_ankle_roll_joint_X4: limit lower=-0.79 upper=0.79 effort=10.5 velocity=8.69 -> lower=-0.79 upper=0.79 effort=28.98 velocity=8.69
- joint left_elbow_pitch_joint_X6: limit lower=-1.31 upper=1.83 effort=20 velocity=16.02 -> lower=-1.31 upper=1.83 effort=23 velocity=16.02
- joint left_hip_pitch_joint_X8: limit lower=-2.53 upper=1.57 effort=43 velocity=13.3 -> lower=-2.53 upper=1.57 effort=72 velocity=13.3
- joint left_hip_roll_joint_X8: limit lower=-0.35 upper=3.14 effort=43 velocity=13.3 -> lower=-0.35 upper=3.14 effort=72 velocity=13.3
- joint left_hip_yaw_joint_X8: limit lower=-1.57 upper=1.57 effort=43 velocity=13.3 -> lower=-1.57 upper=1.57 effort=72 velocity=13.3
- joint left_knee_joint_X8: limit lower=-0.17 upper=1.57 effort=43 velocity=13.3 -> lower=-0.17 upper=1.57 effort=72 velocity=13.3
- joint left_shoulder_pitch_joint_X6: limit lower=-3.02 upper=1.69 effort=20 velocity=16.02 -> lower=-3.02 upper=1.69 effort=23 velocity=16.02
- joint left_shoulder_roll_joint_X6: limit lower=-0.21 upper=2.93 effort=20 velocity=16.02 -> lower=-0.21 upper=2.93 effort=23 velocity=16.02
- joint left_shoulder_yaw_joint_X4: limit lower=-1.75 upper=2.97 effort=10.5 velocity=8.69 -> lower=-1.75 upper=2.97 effort=12.075 velocity=8.69
- joint left_wrist_roll_joint_X4: limit lower=-1.57 upper=1.57 effort=10.5 velocity=8.69 -> lower=-1.57 upper=1.57 effort=12.075 velocity=8.69
- joint left_wrist_yaw_joint_X4: limit lower=-2.36 upper=2.36 effort=10.5 velocity=8.69 -> lower=-2.36 upper=2.36 effort=12.075 velocity=8.69
- joint right_ankle_pitch_joint_X4: limit lower=-0.79 upper=0.79 effort=10.5 velocity=8.69 -> lower=-0.79 upper=0.79 effort=96.6 velocity=8.69
- joint right_ankle_roll_joint_X4: limit lower=-0.79 upper=0.79 effort=10.5 velocity=8.69 -> lower=-0.79 upper=0.79 effort=28.98 velocity=8.69
- joint right_elbow_pitch_joint_X6: limit lower=-1.31 upper=1.83 effort=20 velocity=16.02 -> lower=-1.31 upper=1.83 effort=23 velocity=16.02
- joint right_hip_pitch_joint_X8: limit lower=-2.53 upper=1.57 effort=43 velocity=13.3 -> lower=-2.53 upper=1.57 effort=72 velocity=13.3
- joint right_hip_roll_joint_X8: limit lower=-3.14 upper=0.35 effort=43 velocity=13.3 -> lower=-3.14 upper=0.35 effort=72 velocity=13.3
- joint right_hip_yaw_joint_X8: limit lower=-1.57 upper=1.57 effort=43 velocity=13.3 -> lower=-1.57 upper=1.57 effort=72 velocity=13.3
- joint right_knee_joint_X8: limit lower=-0.17 upper=1.57 effort=43 velocity=13.3 -> lower=-0.17 upper=1.57 effort=72 velocity=13.3
- joint right_shoulder_pitch_joint_X6: limit lower=-3.02 upper=1.69 effort=20 velocity=16.02 -> lower=-3.02 upper=1.69 effort=23 velocity=16.02
- joint right_shoulder_roll_joint_X6: limit lower=-2.93 upper=0.21 effort=20 velocity=16.02 -> lower=-2.93 upper=0.21 effort=23 velocity=16.02
- joint right_shoulder_yaw_joint_X4: limit lower=-2.97 upper=1.75 effort=10.5 velocity=8.69 -> lower=-2.97 upper=1.75 effort=12.075 velocity=8.69
- joint right_wrist_roll_joint_X4: limit lower=-1.57 upper=1.57 effort=10.5 velocity=8.69 -> lower=-1.57 upper=1.57 effort=12.075 velocity=8.69
- joint right_wrist_yaw_joint_X4: limit lower=-2.36 upper=2.36 effort=10.5 velocity=8.69 -> lower=-2.36 upper=2.36 effort=12.075 velocity=8.69
- joint waist_yaw_joint_X8: limit lower=-1.57 upper=1.57 effort=43 velocity=13.3 -> lower=-1.57 upper=1.57 effort=72 velocity=13.3

Commit message: resolve asimetric parts

File: src/control/mc_rtc_controller/urdf/harambe_mc_rtc.urdf (robot description, URDF)
Before this commit: robot harambe_full_robot, 66 links, 65 joints
Joints:
- joint left_hip_pitch_joint_X8: origin xyz=0.0333787 0.076301 -0.467748 rpy=0 0 0 -> xyz=0.0333787 0.072699 -0.467748 rpy=0 0 0
- joint right_ankle_pitch_joint_X4: origin xyz=-4.02748e-07 0.059 -0.395 rpy=0 0 0 -> xyz=-4.02748e-07 0.051 -0.395 rpy=0 0 0
- joint right_hip_roll_joint_X8: origin xyz=0.055 -0.078 0 rpy=0 0 0 -> xyz=0.055 -0.073 0 rpy=0 0 0
