Commit message: harambe v0.4 update

File: src/control/mc_rtc_controller/urdf/harambe_mc_rtc.urdf (robot description, URDF)
Before this commit: robot harambe_full_robot, 66 links, 65 joints
Links:
- removed link left_hand_base_link
- removed link left_index_intermediate
- removed link left_index_proximal
- removed link left_index_tip
- removed link left_middle_intermediate
- removed link left_middle_proximal
- removed link left_middle_tip
- removed link left_pinky_intermediate
- removed link left_pinky_proximal
- removed link left_pinky_tip
- removed link left_ring_intermediate
- removed link left_ring_proximal
- removed link left_ring_tip
- removed link left_thumb_distal
- removed link left_thumb_intermediate
- removed link left_thumb_proximal
- removed link left_thumb_proximal_base
- removed link left_thumb_tip
- removed link right_hand_base_link
- removed link right_index_intermediate
- removed link right_index_proximal
- removed link right_index_tip
- removed link right_middle_intermediate
- removed link right_middle_proximal
- removed link right_middle_tip
- removed link right_pinky_intermediate
- removed link right_pinky_proximal
- removed link right_pinky_tip
- removed link right_ring_intermediate
- removed link right_ring_proximal
- removed link right_ring_tip
- removed link right_thumb_distal
- removed link right_thumb_intermediate
- removed link right_thumb_proximal
- removed link right_thumb_proximal_base
- removed link right_thumb_tip
- link pelvis_imu_sensor: geometry 
- link torso_imu_sensor: geometry 
- link urdf_base: mass 5.132 -> 5.734; geometry collision mesh filename=package://full_robot_description/meshes/collision/b_base.stl; collision mesh filename=package://full_robot_description/meshes/collision/f_base.stl
- link urdf_foot_assembly: mass 0.504 -> 0.309
- link urdf_foot_assembly_2: mass 0.504 -> 0.309
- link urdf_hip_assembly: mass 1.73 -> 1.829
- link urdf_hip_assembly_2: mass 1.73 -> 1.829
- link urdf_l_tibia_assembly: mass 2.4 -> 2.216
- link urdf_l_upper_femur_assembly: mass 1.912 -> 1.93; geometry collision mesh filename=package://full_robot_description/meshes/collision/l_upper_f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; collision mesh filename=package://full_robot_description/meshes/collision/stopper_l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
- link urdf_lower_femur_assembly: mass 1.817 -> 1.832; geometry collision mesh filename=package://full_robot_description/meshes/collision/lower_fem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; collision mesh filename=package://full_robot_description/meshes/collision/stopper_l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
- link urdf_r_tibia_assembly: mass 2.4 -> 2.215
Joints:
- removed joint left_hand_base_joint
- removed joint left_index_intermediate_joint
- removed joint left_index_proximal_joint
- removed joint left_index_tip_joint
- removed joint left_middle_intermediate_joint
- removed joint left_middle_proximal_joint
- removed joint left_middle_tip_joint
- removed joint left_pinky_intermediate_joint
- removed joint left_pinky_proximal_joint
- removed joint left_pinky_tip_joint
- removed joint left_ring_intermediate_joint
- removed joint left_ring_proximal_joint
- removed joint left_ring_tip_joint
- removed joint left_thumb_distal_joint
- removed joint left_thumb_intermediate_joint
- removed joint left_thumb_proximal_pitch_joint
- removed joint left_thumb_proximal_yaw_joint
- removed joint left_thumb_tip_joint
- removed joint right_hand_base_joint
- removed joint right_index_intermediate_joint
- removed joint right_index_proximal_joint
- removed joint right_index_tip_joint
- removed joint right_middle_intermediate_joint
- removed joint right_middle_proximal_joint
- removed joint right_middle_tip_joint
- removed joint right_pinky_intermediate_joint
- removed joint right_pinky_proximal_joint
- removed joint right_pinky_tip_joint
- removed joint right_ring_intermediate_joint
- removed joint right_ring_proximal_joint
- removed joint right_ring_tip_joint
- removed joint right_thumb_distal_joint
- removed joint right_thumb_intermediate_joint
- removed joint right_thumb_proximal_pitch_joint
- removed joint right_thumb_proximal_yaw_joint
- removed joint right_thumb_tip_joint
- joint left_ankle_pitch_joint_X4: limit lower=-0.79 upper=0.79 effort=96.6 velocity=8.69 -> lower=-0.785398 upper=0.785398 effort=10 velocity=10; origin xyz=-1.45092e-06 -0.051 -0.395 rpy=0 0 0 -> xyz=0 -0.051 -0.395 rpy=0 0 0
- joint left_ankle_roll_joint_X4: limit lower=-0.79 upper=0.79 effort=28.98 velocity=8.69 -> lower=-0.785398 upper=0.785398 effort=10 velocity=10; origin xyz=-0.0120001 -0.004 -0.028 rpy=0 0 0 -> xyz=-0.012 -0.004 -0.028 rpy=0 0 0
- joint left_elbow_pitch_joint_X6: limit lower=-1.31 upper=1.83 effort=23 velocity=16.02 -> lower=-1.309 upper=1.8326 effort=10 velocity=10; origin xyz=0.019337 0.0291733 -0.075 rpy=0 -0.0190902 -0.585348 -> xyz=0.0193369 0.0291733 -0.075 rpy=0 -0.0190922 -0.585347
- joint left_hip_pitch_joint_X8: limit lower=-2.53 upper=1.57 effort=72 velocity=13.3 -> lower=-2.61799 upper=2.61799 effort=10 velocity=10; origin xyz=0.0333787 0.072699 -0.467748 rpy=0 0 0 -> xyz=0.070373 0.0872946 -0.431099 rpy=0 0 0
- joint left_hip_roll_joint_X8: limit lower=-0.35 upper=3.14 effort=72 velocity=13.3 -> lower=-0.383972 upper=3.22886 effort=10 velocity=10; origin xyz=0.055 0.073 0 rpy=0 0 0 -> xyz=0.053 0.062 0 rpy=0 0 0
- joint left_hip_yaw_joint_X8: limit lower=-1.57 upper=1.57 effort=72 velocity=13.3 -> lower=-2.15199 upper=2.09003 effort=10 velocity=10; origin xyz=-0.053 -7.97086e-07 -0.217 rpy=0 0 0 -> xyz=-0.053 0 -0.217 rpy=0 0 0
- joint left_knee_joint_X8: limit lower=-0.17 upper=1.57 effort=72 velocity=13.3 -> lower=-1.52716 upper=1.52716 effort=10 velocity=10; origin xyz=0 0.055 -0.113 rpy=0 0 0 -> xyz=-1.45947e-07 0.055 -0.111 rpy=0 0 0
- joint left_shoulder_pitch_joint_X6: limit lower=-3.02 upper=1.69 effort=23 velocity=16.02 -> lower=-3.01942 upper=1.69297 effort=10 velocity=10; origin xyz=0 0.1755 0.423977 rpy=0 0 0 -> xyz=0 0.1695 0.423977 rpy=0 0 0
- joint left_shoulder_roll_joint_X6: limit lower=-0.21 upper=2.93 effort=23 velocity=16.02 -> lower=-0.20944 upper=2.93215 effort=10 velocity=10; origin xyz=0.0456571 0.07 0.00560599 rpy=0 -0.122173 0 -> xyz=0.0456571 0.07 0.00560611 rpy=0 -0.122176 0
- joint left_shoulder_yaw_joint_X4: limit lower=-1.75 upper=2.97 effort=12.075 velocity=8.69 -> lower=-1.74533 upper=2.96706 effort=10 velocity=10; origin xyz=-0.046 0.0343048 -0.161394 rpy=0.209376 0.00530409 -0.0249664 -> xyz=-0.046 0.034306 -0.161394 rpy=0.209383 0.00530439 -0.024967
- joint left_wrist_roll_joint_X4: limit lower=-1.57 upper=1.57 effort=12.075 velocity=8.69 -> lower=-1.5708 upper=1.5708 effort=10 velocity=10; origin xyz=0.0219762 -0.0156859 -0.0615 rpy=-0.248271 0 -0.619909 -> xyz=0.0219762 -0.0156859 -0.0615 rpy=-0.248279 0 -0.619909
- joint left_wrist_yaw_joint_X4: limit lower=-2.36 upper=2.36 effort=12.075 velocity=8.69 -> lower=-2.35619 upper=2.35619 effort=10 velocity=10; origin xyz=0.0391738 -0.035 -0.158223 rpy=-0.142861 -0.19688 0.634041 -> xyz=0.0391735 -0.035 -0.158223 rpy=-0.14286 -0.196878 0.634041
- joint pelvis_imu_joint: origin xyz=0.0735 0.0 -0.17 rpy=0 1.5707963267948966 3.141592653589793 -> xyz=0.1069 -0.0007 -0.4707 rpy=0 1.5707963267948966 3.141592653589793; parent urdf_simplified_torso -> urdf_base
- joint right_ankle_pitch_joint_X4: child urdf_ankle_assembly_2 -> urdf_foot_assembly_2; limit lower=-0.79 upper=0.79 effort=96.6 velocity=8.69 -> lower=-0.785398 upper=0.785398 effort=10 velocity=10; origin xyz=-4.02748e-07 0.051 -0.395 rpy=0 0 0 -> xyz=-0.012 -0.004 -0.028 rpy=0 0 0; parent urdf_r_tibia_assembly -> urdf_ankle_assembly_2
- joint right_ankle_roll_joint_X4: child urdf_foot_assembly_2 -> urdf_ankle_assembly_2; limit lower=-0.79 upper=0.79 effort=28.98 velocity=8.69 -> lower=-0.785398 upper=0.785398 effort=10 velocity=10; origin xyz=-0.012 -0.004 -0.028 rpy=0 0 0 -> xyz=0 0.059 -0.395 rpy=0 0 0; parent urdf_ankle_assembly_2 -> urdf_r_tibia_assembly
- joint right_elbow_pitch_joint_X6: limit lower=-1.31 upper=1.83 effort=23 velocity=16.02 -> lower=-1.309 upper=1.8326 effort=10 velocity=10; origin xyz=0.0220994 -0.0333409 -0.065 rpy=0 -0.019088 0.585341 -> xyz=0.0220994 -0.033341 -0.065 rpy=0 -0.0190815 0.58534
- joint right_hip_pitch_joint_X8: limit lower=-2.53 upper=1.57 effort=72 velocity=13.3 -> lower=-2.61799 upper=2.61799 effort=10 velocity=10; origin xyz=0.0333787 -0.072699 -0.467748 rpy=0 0 0 -> xyz=0.070373 -0.0887054 -0.431099 rpy=0 0 0
- joint right_hip_roll_joint_X8: limit lower=-3.14 upper=0.35 effort=72 velocity=13.3 -> lower=-3.22886 upper=0.383972 effort=10 velocity=10; origin xyz=0.055 -0.073 0 rpy=0 0 0 -> xyz=0.053 -0.062 0 rpy=0 0 0
- joint right_hip_yaw_joint_X8: limit lower=-1.57 upper=1.57 effort=72 velocity=13.3 -> lower=-1.5708 upper=1.5708 effort=10 velocity=10; origin xyz=-0.053 7.97086e-07 -0.217 rpy=0 0 0 -> xyz=-0.053 0 -0.217 rpy=0 0 0
- joint right_knee_joint_X8: limit lower=-0.17 upper=1.57 effort=72 velocity=13.3 -> lower=-1.52716 upper=1.52716 effort=10 velocity=10; origin xyz=0 -0.055 -0.113 rpy=0 0 0 -> xyz=1.45947e-07 -0.055 -0.111 rpy=0 0 0
- joint right_shoulder_pitch_joint_X6: limit lower=-3.02 upper=1.69 effort=23 velocity=16.02 -> lower=-3.01942 upper=1.69297 effort=10 velocity=10; origin xyz=0 -0.1755 0.423977 rpy=0 0 0 -> xyz=0 -0.1695 0.423977 rpy=0 0 0
- joint right_shoulder_roll_joint_X6: limit lower=-2.93 upper=0.21 effort=23 velocity=16.02 -> lower=-2.93215 upper=0.20944 effort=10 velocity=10; origin xyz=0.0456571 -0.07 0.00560599 rpy=0 -0.122173 0 -> xyz=0.0456571 -0.07 0.00560611 rpy=0 -0.122176 0
- joint right_shoulder_yaw_joint_X4: limit lower=-2.97 upper=1.75 effort=12.075 velocity=8.69 -> lower=-2.96706 upper=1.74533 effort=10 velocity=10; origin xyz=-0.046 -0.0353456 -0.166285 rpy=-0.209378 0.00530246 0.0249661 -> xyz=-0.046 -0.0353444 -0.166285 rpy=-0.20937 0.00530239 0.0249667
- joint right_wrist_roll_joint_X4: limit lower=-1.57 upper=1.57 effort=12.075 velocity=8.69 -> lower=-1.65806 upper=1.65806 effort=10 velocity=10; origin xyz=0.0219763 0.0156857 -0.0565 rpy=0.248281 0 0.619897 -> xyz=0.0219763 0.0156857 -0.0565 rpy=0.248276 0 0.619896
- joint right_wrist_yaw_joint_X4: limit lower=-2.36 upper=2.36 effort=12.075 velocity=8.69 -> lower=-2.35619 upper=2.35619 effort=10 velocity=10; origin xyz=0.0403763 0.04 -0.163076 rpy=0.142857 -0.196885 -0.634033 -> xyz=0.0403774 0.04 -0.163076 rpy=0.142861 -0.196891 -0.634034
- joint waist_yaw_joint_X8: limit lower=-1.57 upper=1.57 effort=72 velocity=13.3 -> lower=-2.60054 upper=2.60054 effort=10 velocity=10; origin xyz=0.0333787 -0.000698852 -0.300748 rpy=0 0 0 -> xyz=0.070373 -0.000705351 -0.281099 rpy=0 0 0

Commit message: Dual IMU support, fix right ankle chain, match Isaac Lab physics
- Upgrade observation from 87-dim to 93-dim (dual IMU: pelvis + torso)
- Fix right ankle pitch/roll joint order (was swapped vs Isaac Lab URDF)
- Set joint limits from Isaac Lab URDF (knee [-0.17, 1.57], etc.)
- Set effort limits on MuJoCo actuators (X8=72Nm moderate, ankle_pitch=96.6Nm)
- Set armature to reflected rotor inertia (X8=0.058, X6=0.025, X4=0.039)
- Update PD gains to match Isaac Lab ActuatorCfg
- Add smoothing, clip_actions to GUI for live tuning
- Stiffer ground contact (solref=0.002)
- Fix PelvisIMU parent body (urdf_base, identity rotation)
- Remove joint damping (match Isaac Lab ImplicitActuator)

File: src/control/mc_rtc_controller/urdf/harambe_mc_rtc.urdf (robot description, URDF)
Before this commit: robot robot_harambe_v04, 30 links, 29 joints
Joints:
- joint pelvis_imu_joint: origin xyz=0.1069 -0.0007 -0.4707 rpy=0 1.5707963267948966 3.141592653589793 -> xyz=0.1069 -0.0007 -0.4707 rpy=3.141592653589793 -1.5707963267948966 0
- joint right_ankle_pitch_joint_X4: child urdf_foot_assembly_2 -> urdf_ankle_assembly_2; origin xyz=-0.012 -0.004 -0.028 rpy=0 0 0 -> xyz=0 0.059 -0.395 rpy=0 0 0; parent urdf_ankle_assembly_2 -> urdf_r_tibia_assembly
- joint right_ankle_roll_joint_X4: child urdf_ankle_assembly_2 -> urdf_foot_assembly_2; origin xyz=0 0.059 -0.395 rpy=0 0 0 -> xyz=-0.012 -0.004 -0.028 rpy=0 0 0; parent urdf_r_tibia_assembly -> urdf_ankle_assembly_2
